File: hardware/protopak64.kicad_sch (KiCad schematic)
At the start: 3 parts, among them J1 PakEdge, J2 Breakout2x16

Commit message: Extended hole grid, added second set of headers, and adjusted orientation details.
Parts:
- added J3: Breakout2x16, Connector_PinHeader_2.54mm:PinHeader_2x16_P2.54mm_Vertical, symbol Connector_Generic:Conn_02x16_Odd_Even
Connections:
- net +3V3: now also J3.29 (Pin_29), J3.30 (Pin_30)
- net A0: now also J3.21 (Pin_21)
- net A1: now also J3.19 (Pin_19)
- net A10: now also J3.20 (Pin_20)
- net A11: now also J3.16 (Pin_16)
- net A12: now also J3.5 (Pin_5)
- net A13: now also J3.10 (Pin_10)
- net A14: now also J3.3 (Pin_3)
- net A15: now also J3.6 (Pin_6)
- net A2: now also J3.17 (Pin_17)
- net A3: now also J3.15 (Pin_15)
- net A4: now also J3.13 (Pin_13)
- net A5: now also J3.11 (Pin_11)
- net A6: now also J3.9 (Pin_9)
- net A7: now also J3.7 (Pin_7)
- net A8: now also J3.12 (Pin_12)
- net A9: now also J3.14 (Pin_14)
- net CE: now also J3.4 (Pin_4)
- net D0: now also J3.23 (Pin_23)
- net D1: now also J3.25 (Pin_25)
- net D2: now also J3.31 (Pin_31)
- net D3: now also J3.32 (Pin_32)
- net D4: now also J3.28 (Pin_28)
- net D5: now also J3.26 (Pin_26)
- net D6: now also J3.24 (Pin_24)
- net D7: now also J3.22 (Pin_22)
- net DETECT: now also J3.27 (Pin_27)
- net GND: now also J3.1 (Pin_1), J3.2 (Pin_2)
- net ~{OE}: now also J3.18 (Pin_18)
- net ~{WE}: now also J3.8 (Pin_8)
